Commit message: design v2 dan udah kalibrasi (harusnya)

File: (Unsaved).xacro (robot description, xacro)
@@ -24,10 +24,10 @@
 <link name="teta1_1">
   <inertial>
-    <origin xyz="0.030534126789324406 -0.015667414362937795 -0.00029693086440870514" rpy="0 0 0"/>
+    <origin xyz="0.007457738610655351 -0.033495925310553426 0.0005597644070481703" rpy="0 0 0"/>
     <mass value="0.322485513471676"/>
-    <inertia ixx="7.5e-05" iyy="7.3e-05" izz="9.9e-05" ixy="2e-06" iyz="-0.0" ixz="0.0"/>
-  </inertial>
-  <visual>
-    <origin xyz="0.144694 0.105026 0.0515" rpy="0 0 0"/>
+    <inertia ixx="7.4e-05" iyy="7.3e-05" izz="9.9e-05" ixy="3e-06" iyz="1e-06" ixz="-1e-06"/>
+  </inertial>
+  <visual>
+    <origin xyz="0.114018 0.08132 0.0515" rpy="0 0 0"/>
     <geometry>
       <mesh filename="teta1_1.stl" scale="0.001 0.001 0.001"/>
@@ -36,5 +36,5 @@
   </visual>
   <collision>
-    <origin xyz="0.144694 0.105026 0.0515" rpy="0 0 0"/>
+    <origin xyz="0.114018 0.08132 0.0515" rpy="0 0 0"/>
     <geometry>
       <mesh filename="teta1_1.stl" scale="0.001 0.001 0.001"/>
@@ -44,10 +44,10 @@
 <link name="tibia1_1">
   <inertial>
-    <origin xyz="0.013631914546237855 0.009229301543740576 -0.01387288396315086" rpy="0 0 0"/>
-    <mass value="0.5005531081408956"/>
-    <inertia ixx="0.000169" iyy="0.000166" izz="0.000101" ixy="4e-06" iyz="0.0" ixz="0.0"/>
-  </inertial>
-  <visual>
-    <origin xyz="0.111055 0.154709 0.0515" rpy="0 0 0"/>
+    <origin xyz="0.01300075031251191 0.01014451022429283 -0.01383993691310137" rpy="0 0 0"/>
+    <mass value="0.5005531081408972"/>
+    <inertia ixx="0.000168" iyy="0.000167" izz="0.000102" ixy="5e-06" iyz="-3e-06" ixz="3e-06"/>
+  </inertial>
+  <visual>
+    <origin xyz="0.099235 0.14816 0.049792" rpy="0 0 0"/>
     <geometry>
       <mesh filename="tibia1_1.stl" scale="0.001 0.001 0.001"/>
@@ -56,5 +56,5 @@
   </visual>
   <collision>
-    <origin xyz="0.111055 0.154709 0.0515" rpy="0 0 0"/>
+    <origin xyz="0.099235 0.14816 0.049792" rpy="0 0 0"/>
     <geometry>
       <mesh filename="tibia1_1.stl" scale="0.001 0.001 0.001"/>
@@ -62,12 +62,32 @@
   </collision>
 </link>
+<link name="coxa1_1">
+  <inertial>
+    <origin xyz="0.012623331280600614 -0.014399972809350028 -0.03845464138452408" rpy="0 0 0"/>
+    <mass value="1.0829342534788695"/>
+    <inertia ixx="0.000688" iyy="0.00065" izz="0.000489" ixy="0.000143" iyz="-7.9e-05" ixz="6.9e-05"/>
+  </inertial>
+  <visual>
+    <origin xyz="0.1571 0.05727 -0.0" rpy="0 0 0"/>
+    <geometry>
+      <mesh filename="coxa1_1.stl" scale="0.001 0.001 0.001"/>
+    </geometry>
+    <material name="silver"/>
+  </visual>
+  <collision>
+    <origin xyz="0.1571 0.05727 -0.0" rpy="0 0 0"/>
+    <geometry>
+      <mesh filename="coxa1_1.stl" scale="0.001 0.001 0.001"/>
+    </geometry>
+  </collision>
+</link>
 <link name="teta2_1">
   <inertial>
-    <origin xyz="0.030092369962315096 0.016499999999999838 -0.00029693086440886474" rpy="0 0 0"/>
+    <origin xyz="0.03080650855798238 -0.01509942070888103 0.0009294869219693275" rpy="0 0 0"/>
     <mass value="0.322485513471676"/>
-    <inertia ixx="7.1e-05" iyy="7.6e-05" izz="9.9e-05" ixy="-0.0" iyz="-0.0" ixz="0.0"/>
-  </inertial>
-  <visual>
-    <origin xyz="0.105851 0.0165 0.0515" rpy="0 0 0"/>
+    <inertia ixx="7.1e-05" iyy="7.6e-05" izz="9.9e-05" ixy="-0.0" iyz="-0.0" ixz="-1e-06"/>
+  </inertial>
+  <visual>
+    <origin xyz="0.106659 -0.01862 0.0515" rpy="0 0 0"/>
     <geometry>
       <mesh filename="teta2_1.stl" scale="0.001 0.001 0.001"/>
@@ -76,5 +96,5 @@
   </visual>
   <collision>
-    <origin xyz="0.105851 0.0165 0.0515" rpy="0 0 0"/>
+    <origin xyz="0.106659 -0.01862 0.0515" rpy="0 0 0"/>
     <geometry>
       <mesh filename="teta2_1.stl" scale="0.001 0.001 0.001"/>
@@ -84,10 +104,10 @@
 <link name="tibia2_1">
   <inertial>
-    <origin xyz="2.0452293353345752e-07 0.01646291267745646 -0.013872883963150555" rpy="0 0 0"/>
-    <mass value="0.5005531081408956"/>
-    <inertia ixx="0.000163" iyy="0.000172" izz="0.000101" ixy="0.0" iyz="0.0" ixz="-0.0"/>
-  </inertial>
-  <visual>
-    <origin xyz="0.045851 0.0165 0.0515" rpy="0 0 0"/>
+    <origin xyz="-0.0011772196856956324 0.01642612539978206 -0.013866134636234297" rpy="0 0 0"/>
+    <mass value="0.5005531081408972"/>
+    <inertia ixx="0.000163" iyy="0.000172" izz="0.000101" ixy="-0.0" iyz="0.0" ixz="-2e-06"/>
+  </inertial>
+  <visual>
+    <origin xyz="0.045218 0.011587 0.050239" rpy="0 0 0"/>
     <geometry>
       <mesh filename="tibia2_1.stl" scale="0.001 0.001 0.001"/>
@@ -96,5 +116,5 @@
   </visual>
   <collision>
-    <origin xyz="0.045851 0.0165 0.0515" rpy="0 0 0"/>
+    <origin xyz="0.045218 0.011587 0.050239" rpy="0 0 0"/>
     <geometry>
       <mesh filename="tibia2_1.stl" scale="0.001 0.001 0.001"/>
@@ -102,12 +122,32 @@
   </collision>
 </link>
+<link name="coxa2_1">
+  <inertial>
+    <origin xyz="0.019130272556860894 0.0008632369545831863 -0.03845464138452424" rpy="0 0 0"/>
+    <mass value="1.0829342534788695"/>
+    <inertia ixx="0.000525" iyy="0.000813" izz="0.000489" ixy="-1.3e-05" iyz="5e-06" ixz="0.000105"/>
+  </inertial>
+  <visual>
+    <origin xyz="0.152351 -0.0 -0.0" rpy="0 0 0"/>
+    <geometry>
+      <mesh filename="coxa2_1.stl" scale="0.001 0.001 0.001"/>
+    </geometry>
+    <material name="silver"/>
+  </visual>
+  <collision>
+    <origin xyz="0.152351 -0.0 -0.0" rpy="0 0 0"/>
+    <geometry>
+      <mesh filename="coxa2_1.stl" scale="0.001 0.001 0.001"/>
+    </geometry>
+  </collision>
+</link>
 <link name="teta3_1">
   <inertial>
-    <origin xyz="0.0049988335991379 0.03378988634228103 0.0002969308644092117" rpy="0 0 0"/>
+    <origin xyz="0.03205389994058132 0.011802607043990956 -0.0002969308644088231" rpy="0 0 0"/>
     <mass value="0.322485513471676"/>
-    <inertia ixx="7.4e-05" iyy="7.3e-05" izz="9.9e-05" ixy="-2e-06" iyz="0.0" ixz="0.0"/>
-  </inertial>
-  <visual>
-    <origin xyz="0.115797 -0.084261 0.0515" rpy="0 0 0"/>
+    <inertia ixx="7.4e-05" iyy="7.3e-05" izz="9.9e-05" ixy="-3e-06" iyz="-0.0" ixz="-0.0"/>
+  </inertial>
+  <visual>
+    <origin xyz="0.139127 -0.103221 0.0515" rpy="0 0 0"/>
     <geometry>
       <mesh filename="teta3_1.stl" scale="0.001 0.001 0.001"/>
@@ -116,5 +156,5 @@
   </visual>
   <collision>
-    <origin xyz="0.115797 -0.084261 0.0515" rpy="0 0 0"/>
+    <origin xyz="0.139127 -0.103221 0.0515" rpy="0 0 0"/>
     <geometry>
       <mesh filename="teta3_1.stl" scale="0.001 0.001 0.001"/>
@@ -124,10 +164,10 @@
 <link name="tibia3_1">
   <inertial>
-    <origin xyz="-0.01309616122417527 0.009975931443530317 -0.013872883963150652" rpy="0 0 0"/>
-    <mass value="0.5005531081408956"/>
-    <inertia ixx="0.000169" iyy="0.000166" izz="0.000101" ixy="-4e-06" iyz="0.0" ixz="-0.0"/>
-  </inertial>
-  <visual>
-    <origin xyz="0.079437 -0.13199 0.0515" rpy="0 0 0"/>
+    <origin xyz="-0.012443498606944797 0.010778592092196643 -0.013872883963235084" rpy="0 0 0"/>
+    <mass value="0.5005531081408972"/>
+    <inertia ixx="0.000168" iyy="0.000167" izz="0.000101" ixy="-4e-06" iyz="0.0" ixz="-0.0"/>
+  </inertial>
+  <visual>
+    <origin xyz="0.074899 -0.126966 0.0515" rpy="0 0 0"/>
     <geometry>
       <mesh filename="tibia3_1.stl" scale="0.001 0.001 0.001"/>
@@ -136,5 +176,5 @@
   </visual>
   <collision>
-    <origin xyz="0.079437 -0.13199 0.0515" rpy="0 0 0"/>
+    <origin xyz="0.074899 -0.126966 0.0515" rpy="0 0 0"/>
     <geometry>
       <mesh filename="tibia3_1.stl" scale="0.001 0.001 0.001"/>
@@ -142,12 +182,32 @@
   </collision>
 </link>
+<link name="coxa3_1">
+  <inertial>
+    <origin xyz="0.012550506304740416 0.01446349281278922 -0.038454641384523994" rpy="0 0 0"/>
+    <mass value="1.0829342534788695"/>
+    <inertia ixx="0.000689" iyy="0.000649" izz="0.000489" ixy="-0.000143" iyz="7.9e-05" ixz="6.9e-05"/>
+  </inertial>
+  <visual>
+    <origin xyz="0.1571 -0.05727 -0.0" rpy="0 0 0"/>
+    <geometry>
+      <mesh filename="coxa3_1.stl" scale="0.001 0.001 0.001"/>
+    </geometry>
+    <material name="silver"/>
+  </visual>
+  <collision>
+    <origin xyz="0.1571 -0.05727 -0.0" rpy="0 0 0"/>
+    <geometry>
+      <mesh filename="coxa3_1.stl" scale="0.001 0.001 0.001"/>
+    </geometry>
+  </collision>
+</link>
 <link name="teta4_1">
   <inertial>
-    <origin xyz="-0.031894846797939025 0.012668757983660323 -0.00029693086440856636" rpy="0 0 0"/>
+    <origin xyz="-0.007231179844230107 0.033548934178161266 -0.0002969308644086843" rpy="0 0 0"/>
     <mass value="0.322485513471676"/>
     <inertia ixx="7.4e-05" iyy="7.3e-05" izz="9.9e-05" ixy="3e-06" iyz="0.0" ixz="-0.0"/>
   </inertial>
   <visual>
-    <origin xyz="0.254528 -0.103617 0.0515" rpy="0 0 0"/>
+    <origin xyz="0.280518 -0.081614 0.0515" rpy="0 0 0"/>
     <geometry>
       <mesh filename="teta4_1.stl" scale="0.001 0.001 0.001"/>
@@ -156,5 +216,5 @@
   </visual>
   <collision>
-    <origin xyz="0.254528 -0.103617 0.0515" rpy="0 0 0"/>
+    <origin xyz="0.280518 -0.081614 0.0515" rpy="0 0 0"/>
     <geometry>
       <mesh filename="teta4_1.stl" scale="0.001 0.001 0.001"/>
@@ -164,10 +224,10 @@
 <link name="tibia4_1">
   <inertial>
-    <origin xyz="-0.01268524175515362 -0.010494219075531164 -0.013872883963149903" rpy="0 0 0"/>
-    <mass value="0.5005531081408956"/>
+    <origin xyz="-0.012444027191681306 -0.010778842746671374 -0.013872883963234932" rpy="0 0 0"/>
+    <mass value="0.5005531081408972"/>
     <inertia ixx="0.000168" iyy="0.000167" izz="0.000101" ixy="4e-06" iyz="-0.0" ixz="-0.0"/>
   </inertial>
   <visual>
-    <origin xyz="0.292773 -0.149848 0.0515" rpy="0 0 0"/>
+    <origin xyz="0.294859 -0.148572 0.0515" rpy="0 0 0"/>
     <geometry>
       <mesh filename="tibia4_1.stl" scale="0.001 0.001 0.001"/>
@@ -176,5 +236,5 @@
   </visual>
   <collision>
-    <origin xyz="0.292773 -0.149848 0.0515" rpy="0 0 0"/>
+    <origin xyz="0.294859 -0.148572 0.0515" rpy="0 0 0"/>
     <geometry>
       <mesh filename="tibia4_1.stl" scale="0.001 0.001 0.001"/>
@@ -182,12 +242,32 @@
   </collision>
 </link>
+<link name="coxa4_1">
+  <inertial>
+    <origin xyz="-0.012525182858772466 0.014485940570305444 -0.03845464138452389" rpy="0 0 0"/>
+    <mass value="1.0829342534788695"/>
+    <inertia ixx="0.00069" iyy="0.000648" izz="0.000489" ixy="0.000143" iyz="8e-05" ixz="-6.9e-05"/>
+  </inertial>
+  <visual>
+    <origin xyz="0.237601 -0.05727 -0.0" rpy="0 0 0"/>
+    <geometry>
+      <mesh filename="coxa4_1.stl" scale="0.001 0.001 0.001"/>
+    </geometry>
+    <material name="silver"/>
+  </visual>
+  <collision>
+    <origin xyz="0.237601 -0.05727 -0.0" rpy="0 0 0"/>
+    <geometry>
+      <mesh filename="coxa4_1.stl" scale="0.001 0.001 0.001"/>
+    </geometry>
+  </collision>
+</link>
 <link name="teta5_1">
   <inertial>
-    <origin xyz="-0.03009196091642463 -0.016500000000000042 -0.00029693086440888555" rpy="0 0 0"/>
+    <origin xyz="-0.03014949429074193 0.016394643449314152 -0.0002969308644087121" rpy="0 0 0"/>
     <mass value="0.322485513471676"/>
     <inertia ixx="7.1e-05" iyy="7.6e-05" izz="9.9e-05" ixy="-0.0" iyz="-0.0" ixz="-0.0"/>
   </inertial>
   <visual>
-    <origin xyz="0.288851 -0.0165 0.0515" rpy="0 0 0"/>
+    <origin xyz="0.288793 0.016662 0.0515" rpy="0 0 0"/>
     <geometry>
       <mesh filename="teta5_1.stl" scale="0.001 0.001 0.001"/>
@@ -196,5 +276,5 @@
   </visual>
   <collision>
-    <origin xyz="0.288851 -0.0165 0.0515" rpy="0 0 0"/>
+    <origin xyz="0.288793 0.016662 0.0515" rpy="0 0 0"/>
     <geometry>
       <mesh filename="teta5_1.stl" scale="0.001 0.001 0.001"/>
@@ -202,12 +282,72 @@
   </collision>
 </link>
+<link name="tibia6_1">
+  <inertial>
+    <origin xyz="5.772391614522476e-05 -0.016462667283913355 -0.013872883963234946" rpy="0 0 0"/>
+    <mass value="0.5005531081408972"/>
+    <inertia ixx="0.000163" iyy="0.000172" izz="0.000101" ixy="-0.0" iyz="-0.0" ixz="0.0"/>
+  </inertial>
+  <visual>
+    <origin xyz="0.348908 -0.016128 0.0515" rpy="0 0 0"/>
+    <geometry>
+      <mesh filename="tibia6_1.stl" scale="0.001 0.001 0.001"/>
+    </geometry>
+    <material name="silver"/>
+  </visual>
+  <collision>
+    <origin xyz="0.348908 -0.016128 0.0515" rpy="0 0 0"/>
+    <geometry>
+      <mesh filename="tibia6_1.stl" scale="0.001 0.001 0.001"/>
+    </geometry>
+  </collision>
+</link>
+<link name="coxa5_1">
+  <inertial>
+    <origin xyz="-0.01914926572398204 -4.970195210862727e-05 -0.038454641384523945" rpy="0 0 0"/>
+    <mass value="1.0829342534788695"/>
+    <inertia ixx="0.000525" iyy="0.000813" izz="0.000489" ixy="-0.0" iyz="-0.0" ixz="-0.000105"/>
+  </inertial>
+  <visual>
+    <origin xyz="0.242351 -0.0 -0.0" rpy="0 0 0"/>
+    <geometry>
+      <mesh filename="coxa5_1.stl" scale="0.001 0.001 0.001"/>
+    </geometry>
+    <material name="silver"/>
+  </visual>
+  <collision>
+    <origin xyz="0.242351 -0.0 -0.0" rpy="0 0 0"/>
+    <geometry>
+      <mesh filename="coxa5_1.stl" scale="0.001 0.001 0.001"/>
+    </geometry>
+  </collision>
+</link>
+<link name="teta6_1">
+  <inertial>
+    <origin xyz="-0.03217417984423032 -0.011941934178161306 -0.0002969308644086427" rpy="0 0 0"/>
+    <mass value="0.322485513471676"/>
+    <inertia ixx="7.4e-05" iyy="7.3e-05" izz="9.9e-05" ixy="-3e-06" iyz="-0.0" ixz="-0.0"/>
+  </inertial>
+  <visual>
+    <origin xyz="0.255575 0.103221 0.0515" rpy="0 0 0"/>
+    <geometry>
+      <mesh filename="teta6_1.stl" scale="0.001 0.001 0.001"/>
+    </geometry>
+    <material name="silver"/>
+  </visual>
+  <collision>
+    <origin xyz="0.255575 0.103221 0.0515" rpy="0 0 0"/>
+    <geometry>
+      <mesh filename="teta6_1.stl" scale="0.001 0.001 0.001"/>
+    </geometry>
+  </collision>
+</link>
 <link name="tibia5_1">
   <inertial>
-    <origin xyz="2.0452295651507413e-07 -0.01646291267745669 -0.013872883963150527" rpy="0 0 0"/>
-    <mass value="0.5005531081408956"/>
-    <inertia ixx="0.000163" iyy="0.000172" izz="0.000101" ixy="0.0" iyz="-0.0" ixz="0.0"/>
-  </inertial>
-  <visual>
-    <origin xyz="0.348851 -0.0165 0.0515" rpy="0 0 0"/>
+    <origin xyz="0.012443907652835318 -0.010778592092196587 -0.013872883963234918" rpy="0 0 0"/>
+    <mass value="0.5005531081408972"/>
+    <inertia ixx="0.000168" iyy="0.000167" izz="0.000101" ixy="-4e-06" iyz="-0.0" ixz="0.0"/>
+  </inertial>
+  <visual>
+    <origin xyz="0.319803 0.126966 0.0515" rpy="0 0 0"/>
     <geometry>
       <mesh filename="tibia5_1.stl" scale="0.001 0.001 0.001"/>
@@ -216,5 +356,5 @@
   </visual>
   <collision>
-    <origin xyz="0.348851 -0.0165 0.0515" rpy="0 0 0"/>
+    <origin xyz="0.319803 0.126966 0.0515" rpy="0 0 0"/>
     <geometry>
       <mesh filename="tibia5_1.stl" scale="0.001 0.001 0.001"/>
@@ -222,149 +362,9 @@
   </collision>
 </link>
-<link name="teta6_1">
-  <inertial>
-    <origin xyz="-0.004160848120962735 -0.034065716062035664 -0.00029693086440885086" rpy="0 0 0"/>
-    <mass value="0.322485513471676"/>
-    <inertia ixx="7.5e-05" iyy="7.3e-05" izz="9.9e-05" ixy="-2e-06" iyz="-0.0" ixz="-0.0"/>
-  </inertial>
-  <visual>
-    <origin xyz="0.278135 0.085404 0.0515" rpy="0 0 0"/>
-    <geometry>
-      <mesh filename="teta6_1.stl" scale="0.001 0.001 0.001"/>
-    </geometry>
-    <material name="silver"/>
-  </visual>
-  <collision>
-    <origin xyz="0.278135 0.085404 0.0515" rpy="0 0 0"/>
-    <geometry>
-      <mesh filename="teta6_1.stl" scale="0.001 0.001 0.001"/>
-    </geometry>
-  </collision>
-</link>
-<link name="tibia6_1">
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